Commit message: Update models file

File: models/pioneer3dx.urdf (robot description, URDF)
Before this commit: robot /home/leanhchien/webots_ws/src/pioneer3dx/resource/pioneer3dx.urdf, 10 links, 9 joints
Links:
- added link map
Joints:
- added joint base_map: type fixed, parent world, child map, origin xyz=-15.0 -15.0 0.0 rpy=0 0 0
- joint base_link_lidar_joint: origin xyz=0.1 0 0.19 rpy=0 0 0 -> xyz=0 0 0.19 rpy=0 0 0
